Commit message: base_link to chassis

File: urdf/gazebo_control.xacro (robot description, xacro)
@@ -5,6 +5,6 @@
             filename="libgz-sim-diff-drive-system.so"
             name="gz::sim::systems::DiffDrive">
-            <left_joint>base_link_to_lf_wheel</left_joint>
-            <right_joint>base_link_to_rf_wheel</right_joint>
+            <left_joint>chassis_to_lf_wheel</left_joint>
+            <right_joint>chassis_to_rf_wheel</right_joint>
             <wheel_separation>0.3</wheel_separation>
             <wheel_radius>0.06</wheel_radius>
@@ -14,5 +14,5 @@
             <odom_publish_frequency>50</odom_publish_frequency>
             <odom_frame>odom</odom_frame>
-            <base_frame>base_link</base_frame>
+            <base_frame>chassis</base_frame>
             <publish_odom>true</publish_odom>
             <publish_odom_tf>true</publish_odom_tf>

File: urdf/goal_e.urdf.xacro (robot description, xacro)
@@ -2,4 +2,5 @@
 <robot xmlns:xacro="http://www.ros.org/wiki/xacro" name="myfirst_xacro">
     <xacro:include filename="ros2_control.xacro" />
+    <!-- <xacro:include filename="lidar.xacro" /> -->
     <!-- <xacro:include filename="gazebo_control.xacro" /> -->
     <!-- Parameters -->
@@ -22,4 +23,11 @@
     <xacro:property name="omni_z" value="${base_to_ground - (base_height/2) - omni_wheel_radius}" />
     <link name="base_link">
+    </link>
+    <joint name="chassis_joint" type="fixed">
+        <parent link="base_link" />
+        <child link="chassis" />
+        <origin xyz="-0 0 0" />
+    </joint>
+    <link name="chassis">
         <visual>
             <geometry>
@@ -83,21 +91,4 @@
         </joint>
     </xacro:macro>
-    <!-- Omni Wheel Macro -->
-    <xacro:macro name="omniWheel" params="name parent x y z rpy">
-        <link name="${name}">
-            <visual>
-                <geometry>
-                    <sphere radius="${omni_wheel_radius}" />
-                </geometry>
-                <origin xyz="0 0 ${-omni_z}" />
-            </visual>
-        </link>
-        <joint name="${parent}_to_${name}" type="continuous">
-            <parent link="${parent}" />
-            <child link="${name}" />
-            <origin xyz="${x} ${y} ${z}" rpy="${rpy}" />
-            <axis xyz="0 0 1" />
-        </joint>
-    </xacro:macro>
     <!-- Lidar Macro -->
     <xacro:macro name="lidar" params="name parent x y z rpy">
@@ -138,5 +129,5 @@
     <!-- Wheels -->
     <xacro:wheel name="lb_wheel"
-        parent="base_link"
+        parent="chassis"
         x="${-wheel_offset_x}"
         y="${wheel_offset_y}"
@@ -145,5 +136,5 @@
         axs="0 0 1" />
     <xacro:wheel name="rb_wheel"
-        parent="base_link"
+        parent="chassis"
         x="${-wheel_offset_x}"
         y="${-wheel_offset_y}"
@@ -152,5 +143,5 @@
         axs="0 0 -1" />
     <xacro:wheel name="lf_wheel"
-        parent="base_link"
+        parent="chassis"
         x="${+wheel_offset_x}"
         y="${wheel_offset_y}"
@@ -159,5 +150,5 @@
         axs="0 0 1" />
     <xacro:wheel name="rf_wheel"
-        parent="base_link"
+        parent="chassis"
         x="${+wheel_offset_x}"
         y="${-wheel_offset_y}"
@@ -167,5 +158,5 @@
     <!-- Lidar -->
     <xacro:lidar name="lidar1"
-        parent="base_link"
+        parent="chassis"
         x="0.1"
         y="0"

File: urdf/ros2_control.xacro (robot description, xacro)
@@ -5,5 +5,5 @@
             <plugin>gz_ros2_control/GazeboSimSystem</plugin>
         </hardware>
-        <joint name="base_link_to_lf_wheel">
+        <joint name="chassis_to_lf_wheel">
             <command_interface name="velocity">
                 <param name="min">-10</param>
@@ -13,5 +13,5 @@
             <state_interface name="position" />
         </joint>
-        <joint name="base_link_to_rf_wheel">
+        <joint name="chassis_to_rf_wheel">
             <command_interface name="velocity">
                 <param name="min">-10</param>
@@ -21,5 +21,5 @@
             <state_interface name="position" />
         </joint>
-        <joint name="base_link_to_lb_wheel">
+        <joint name="chassis_to_lb_wheel">
             <command_interface name="velocity">
                 <param name="min">-10</param>
@@ -29,5 +29,5 @@
             <state_interface name="position" />
         </joint>
-        <joint name="base_link_to_rb_wheel">
+        <joint name="chassis_to_rb_wheel">
             <command_interface name="velocity">
                 <param name="min">-10</param>
