Commit message: map init

File: urdf/goal_e.urdf.xacro (robot description, xacro)
@@ -22,4 +22,11 @@
     <xacro:property name="omni_z" value="${base_to_ground - (base_height/2) - omni_wheel_radius}" />
     <link name="base_link">
+    </link>
+    <joint name="base_footprint_joint" type="fixed">
+        <parent link="base_link" />
+        <child link="base_footprint" />
+        <origin xyz="0 0 0" rpy="0 0 0" />
+    </joint>
+    <link name="base_footprint">
     </link>
     <joint name="chassis_joint" type="fixed">

Commit message: turning fix - friction

File: urdf/goal_e.urdf.xacro (robot description, xacro)
@@ -7,5 +7,5 @@
     <xacro:property name="base_width" value="0.3" />
     <xacro:property name="base_height" value="0.1" />
-    <xacro:property name="base_mass" value="1" />
+    <xacro:property name="base_mass" value="5" />
     <xacro:property name="wheel_radius" value="0.06" />
     <xacro:property name="wheel_width" value="0.05" />
@@ -90,4 +90,9 @@
             </inertial>
         </link>
+        <gazebo reference="${name}">
+            <mu1>1.0</mu1>
+            <mu2>0.4</mu2>
+            <fdir1>1 0 0</fdir1>
+        </gazebo>
         <joint name="${parent}_to_${name}" type="continuous">
             <parent link="${parent}" />

Commit message: arm control

File: urdf/goal_e.urdf.xacro (robot description, xacro)
@@ -15,4 +15,9 @@
     <xacro:property name="lidar_width" value="0.03" />
     <xacro:property name="lidar_mass" value="0.1" />
+    <xacro:property name="arm_vert_length" value="0.3" />
+    <xacro:property name="arm_vert_radius" value="0.01" />
+    <xacro:property name="arm_horiz_length" value="${base_width*0.4}" />
+    <xacro:property name="arm_horiz_radius" value="0.01" />
+    <xacro:property name="arm_mass" value="0.4" />
     <!-- Derived -->
     <xacro:property name="base_to_ground" value="${wheel_radius + base_height/2}" />
@@ -168,4 +173,62 @@
         </gazebo>
     </xacro:macro>
+    <!-- L-Shaped Arm Macro -->
+    <xacro:macro name="arm_L" params="name parent x y z rpy axis dir=1">
+        <link name="${name}">
+            <!-- Vertical segment -->
+            <visual>
+                <geometry>
+                    <cylinder length="${arm_vert_length}" radius="${arm_vert_radius}" />
+                </geometry>
+                <origin xyz="0 0 ${arm_vert_length/2}" />
+                <material name="black">
+                    <color rgba="0 0 0 1.0" />
+                </material>
+            </visual>
+            <!-- Horizontal segment -->
+            <visual>
+                <geometry>
+                    <cylinder length="${arm_horiz_length}" radius="${arm_horiz_radius}" />
+                </geometry>
+                <origin xyz="0 ${dir * arm_horiz_length/2} ${arm_vert_length}"
+                    rpy="1.5708 0 0" />
+                <material name="black">
+                    <color rgba="0 0 0 1.0" />
+                </material>
+            </visual>
+            <!-- Collisions -->
+            <collision>
+                <geometry>
+                    <cylinder length="${arm_vert_length}" radius="${arm_vert_radius}" />
+                </geometry>
+                <origin xyz="0 0 ${arm_vert_length/2}" />
+            </collision>
+            <collision>
+                <geometry>
+                    <cylinder length="${arm_horiz_length}" radius="${arm_horiz_radius}" />
+                </geometry>
+                <origin xyz="0 ${dir * arm_horiz_length/2} ${arm_vert_length}"
+                    rpy="1.5708 0 0" />
+            </collision>
+            <!-- Inertial -->
+            <inertial>
+                <mass value="${arm_mass}" />
+                <origin xyz="0 0 ${arm_vert_length/2}" />
+                <inertia
+                    ixx="${(1.0/12.0)*arm_mass*(3*arm_vert_radius*arm_vert_radius + arm_vert_length*arm_vert_length)}"
+                    iyy="${(1.0/12.0)*arm_mass*(3*arm_vert_radius*arm_vert_radius + arm_vert_length*arm_vert_length)}"
+                    izz="${0.5 * arm_mass * arm_vert_radius * arm_vert_radius}"
+                    ixy="0" ixz="0" iyz="0"
+                />
+            </inertial>
+        </link>
+        <!-- Joint -->
+        <joint name="${parent}_to_${name}" type="continuous">
+            <parent link="${parent}" />
+            <child link="${name}" />
+            <origin xyz="${x} ${y} ${z}" rpy="${rpy}" />
+            <axis xyz="${axis}" />
+        </joint>
+    </xacro:macro>
     <!-- Wheels -->
     <xacro:wheel name="lb_wheel"
@@ -204,3 +267,20 @@
         z="${base_height/2}"
         rpy="0 0 0" />
+    <xacro:arm_L
+        name="arm1"
+        parent="chassis"
+        x="${base_length/2}" y="${base_width/2 - arm_vert_radius}"
+        z="${-(base_height/2 - arm_vert_radius)}"
+        rpy="0 1.5708 0"
+        axis="0 0 1"
+        dir="-1"
+    />
+    <xacro:arm_L
+        name="arm2"
+        parent="chassis"
+        x="${base_length/2}" y="${-(base_width/2 - arm_vert_radius)}"
+        z="${-(base_height/2 - arm_vert_radius)}"
+        rpy="0 1.5708 0"
+        axis="0 0 1"
+    />
 </robot>

File: urdf/ros2_control.xacro (robot description, xacro)
@@ -37,4 +37,14 @@
             <state_interface name="position" />
         </joint>
+        <joint name="chassis_to_arm1">
+            <command_interface name="position" />
+            <state_interface name="position" />
+            <state_interface name="velocity" />
+        </joint>
+        <joint name="chassis_to_arm2">
+            <command_interface name="position" />
+            <state_interface name="position" />
+            <state_interface name="velocity" />
+        </joint>
     </ros2_control>
     <gazebo>

Commit message: tragectory controller

File: urdf/goal_e.urdf.xacro (robot description, xacro)
@@ -4,6 +4,6 @@
     <!-- <xacro:include filename="gazebo_control.xacro" /> -->
     <!-- Parameters -->
-    <xacro:property name="base_length" value="0.5" />
-    <xacro:property name="base_width" value="0.3" />
+    <xacro:property name="base_length" value="0.6" />
+    <xacro:property name="base_width" value="0.6" />
     <xacro:property name="base_height" value="0.1" />
     <xacro:property name="base_mass" value="5" />
@@ -15,5 +15,5 @@
     <xacro:property name="lidar_width" value="0.03" />
     <xacro:property name="lidar_mass" value="0.1" />
-    <xacro:property name="arm_vert_length" value="0.3" />
+    <xacro:property name="arm_vert_length" value="0.5" />
     <xacro:property name="arm_vert_radius" value="0.01" />
     <xacro:property name="arm_horiz_length" value="${base_width*0.4}" />
@@ -73,5 +73,5 @@
                     <cylinder length="${wheel_width}" radius="${wheel_radius}" />
                 </geometry>
-                <origin xyz="0 0 ${wheel_width/2}" />
+                <origin xyz="0 -0.005 ${wheel_width/2}" />
                 <material name="black">
                     <color rgba="0.0 0.0 0.0 1.0" />
@@ -163,5 +163,5 @@
                     </scan>
                     <range>
-                        <min>0.08</min>
+                        <min>0.72</min>
                         <max>10.0</max>
                         <resolution>0.01</resolution>
@@ -263,5 +263,5 @@
     <xacro:lidar name="lidar1"
         parent="chassis"
-        x="0.1"
+        x="0.15"
         y="0"
         z="${base_height/2}"

Commit message: 3 goal

File: urdf/goal_e.urdf.xacro (robot description, xacro)
@@ -7,5 +7,5 @@
     <xacro:property name="base_width" value="0.6" />
     <xacro:property name="base_height" value="0.1" />
-    <xacro:property name="base_mass" value="5" />
+    <xacro:property name="base_mass" value="2" />
     <xacro:property name="wheel_radius" value="0.06" />
     <xacro:property name="wheel_width" value="0.05" />
@@ -19,5 +19,5 @@
     <xacro:property name="arm_horiz_length" value="${base_width*0.4}" />
     <xacro:property name="arm_horiz_radius" value="0.01" />
-    <xacro:property name="arm_mass" value="0.4" />
+    <xacro:property name="arm_mass" value="0.01" />
     <!-- Derived -->
     <xacro:property name="base_to_ground" value="${wheel_radius + base_height/2}" />
